File: Adafruit Ultimate GPS.brd (EAGLE design)
At the start: 22.9 x 35.3 mm, 20 parts, among them U1 FGPMMOPA6B, U2 RT9193-3.3

Commit message: v3!
Parts:
- removed RTC: (no value), microbuilder:SOLDERJUMPER_CLOSEDWIRE
- removed U$16: (no value), microbuilder:ADAFRUIT_TEXT_20MM
- added U$20: U.FL, microbuilder:U.FL
- JP1: device microbuilder:1X08_ROUND_70 -> microbuilder:1X09_ROUND_70
- U1: value FGPMMOPA6B -> FGPMMOPA6H; device microbuilder:FGPMMOPA6B -> microbuilder:FGPMMOPA6H
- moved R1 19.4 mm to (2.13, 17.9), turned to 90 degrees
- moved LED1 18.5 mm to (2.18, 22.0), turned to 180 degrees
- moved FID1 16.0 mm to (18.7, 22.5)
- moved FID2 13.5 mm to (2.18, 12.4)
- moved U$15 4.01 mm to (7.49, 26.9)
- moved R3 3.91 mm to (23.7, 10.4), turned to 90 degrees
- moved C1 3.87 mm to (22.0, 24.9)
- moved R2 3.78 mm to (22.0, 20.8)
- moved U1 3.64 mm to (12.2, 17.5)
- moved C2 3.52 mm to (24.0, 24.9)
- moved FB1 3.42 mm to (24.0, 20.8)
- moved U2 3.42 mm to (23.0, 17.2)
- moved C3 3.37 mm to (23.0, 14.6)
- moved D1 3.24 mm to (21.8, 10.8), turned to 270 degrees
- moved U$9 2.90 mm to (22.9, 31.4)
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Connections:
- new net 1PPS: JP1.1, U1.P$13
- new net N$4: U$20.P$3, U1.P$11
- net 3.3V: now also JP1.9; no longer JP1.8, RTC.2
- net ENABLE: now also JP1.8; no longer JP1.7
- net FIX: now also JP1.6; no longer JP1.5
- net GND: now also JP1.3, U$20.P$1, U$20.P$2, U1.P$12, U1.P$19; no longer JP1.2
- net RX_5V: now also JP1.4; no longer JP1.3
- net TX: now also JP1.5; no longer JP1.4
- net VBACKUP: now also JP1.7; no longer JP1.6, RTC.1
- net VIN: now also JP1.2; no longer JP1.1
Routing:
- net 1PPS: track 0.00 -> 28.7 mm, vias 0 -> 1
- net FIX: track 55.4 -> 29.1 mm
- net VBACKUP: track 48.2 -> 34.1 mm, vias 2 -> 1
- net ENABLE: track 30.4 -> 39.0 mm
- net VIN: track 19.0 -> 25.3 mm, vias 1 -> 2
- net GND: track 38.3 -> 43.1 mm, vias 5 -> 8
- net N$4: track 0.00 -> 1.90 mm
- net TX: track 8.93 -> 10.5 mm
- net 3.3V: track 60.6 -> 59.2 mm, vias 0 -> 3
- net RX_5V: track 11.2 -> 12.4 mm
- net RX: track 5.36 -> 6.54 mm
Other:
- board size 22.9 x 35.3 mm -> 25.5 x 33.9 mm
- board text added: "Breakout v3"
- board text added: "PPS"
- board text removed: "Breakout"
- board text removed: "Cut RTC to"
- board text removed: "RTC"
- board text removed: "enable CR1220"

Commit message: updated!
Parts:
- added D2: CUS520, microbuilder:SOD-323
- added U$16: (no value), microbuilder:PCBFEAT-REV-040
- added U$18: (no value), microbuilder:ADAFRUIT_5MM
- C1, C2, C3, FB1, R1, R2, R3: device microbuilder:0805 -> microbuilder:0805-NO
- D1: device adafruit:SOD-323F -> microbuilder:SOD-323
- LED1: value FIX -> RED
- U$8, U$9: value MOUNTINGHOLE2.0 -> MOUNTINGHOLE2.5; device microbuilder:MOUNTINGHOLE_2.0_PLATED -> microbuilder:MOUNTINGHOLE_2.5_PLATED
- U2: value RT9193-3.3 -> MIC5225-3.3
- moved FID1 8.33 mm to (24.1, 28.8)
- moved U$15 4.13 mm to (11.5, 27.9)
- moved FID2 2.73 mm to (2.06, 9.63)
- moved U$20 0.51 mm to (18.9, 29.0)
- moved U$8 0.36 mm to (2.54, 31.8)
- moved U$9 0.36 mm to (22.9, 31.8)
- moved U2 0.25 mm to (23.0, 17.0)
- moved C3 0.25 mm to (23.0, 14.3)
- turned D1 to 90 degrees
Connections:
- removed net RX_5V: D1.C, JP1.4
- new net N$1: B1.+$1, B1.+$2, D2.A
- new net RX_3V: D1.A, R3.2, U1.P$10
- net RX: now also D1.C, JP1.4; no longer D1.A, R3.2, U1.P$10
- net VBACKUP: now also D2.C; no longer B1.+$1
Routing:
- net N$1: track 0.00 -> 41.3 mm, vias 0 -> 1
- net GND: track 43.1 -> 25.0 mm, vias 8 -> 44
- net RX_5V: track 12.4 -> 0.00 mm
- net VBACKUP: track 34.1 -> 23.5 mm
- net RX_3V: track 0.00 -> 7.25 mm
- net RX: track 6.54 -> 12.2 mm
- net 3.3V: track 59.2 -> 55.7 mm
- net 1PPS: track 28.7 -> 26.4 mm
- net VIN: track 25.3 -> 23.1 mm
- net ENABLE: track 39.0 -> 37.9 mm
- net FIX: track 29.1 -> 30.0 mm
- net N$4: track 1.90 -> 2.55 mm
- added copper zone on layer 1, net GND
Other:
- board size 25.5 x 33.9 mm -> 25.4 x 34.3 mm
