File: Adafruit Ultimate GPS.sch (EAGLE design)
At the start: 18 parts, among them U1 FGPMMOPA6B, U2 RT9193-3.3

Commit message: v3!
Parts:
- removed RTC: (no value), microbuilder:SOLDERJUMPER_CLOSED
- added U$20: U.FL, microbuilder:U.FL
- JP1: device microbuilder:HEADER-1X870MIL -> microbuilder:HEADER-1X970MIL
- U1: value FGPMMOPA6B -> FGPMMOPA6H; device microbuilder:GPS_FGPMMOPA6B -> microbuilder:GPS_FGPMMOPA6H
Connections:
- new net 1PPS: JP1.1, U1.1PPS
- new net N$4: U$20.SIGNAL, U1.EX_ANT
- net 3.3V: now also JP1.9; no longer JP1.8, RTC.2
- net ENABLE: now also JP1.8; no longer JP1.7
- net FIX: now also JP1.6; no longer JP1.5
- net GND: now also JP1.3, U$20.GND@0, U$20.GND@1, U1.GND@3, U1.GND@4; no longer JP1.2
- net RX_5V: now also JP1.4; no longer JP1.3
- net TX: now also JP1.5; no longer JP1.4
- net VBACKUP: now also JP1.7; no longer JP1.6, RTC.1
- net VIN: now also JP1.2; no longer JP1.1
Other:
- moved on the sheet: B1
Changed lines of the file:
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@@
 <parts>
 <part name="U$1" library="microbuilder" deviceset="FRAME_A4_ADAFRUIT" device=""/>
-<part name="U1" library="microbuilder" deviceset="GPS_FGPMMOPA6B" device="" value="FGPMMOPA6B"/>
+<part name="U1" library="microbuilder" deviceset="GPS_FGPMMOPA6H" device="" value="FGPMMOPA6H"/>
 <part name="U2" library="microbuilder" deviceset="VREG_SOT23-5" device="" value="RT9193-3.3"/>
 <part name="LED1" library="microbuilder" deviceset="LED" device="0805" value="FIX"/>
@@
 <part name="U$8" library="microbuilder" deviceset="MOUNTINGHOLE" device="2.0"/>
 <part name="U$9" library="microbuilder" deviceset="MOUNTINGHOLE" device="2.0"/>
-<part name="JP1" library="microbuilder" deviceset="HEADER-1X8" device="70MIL"/>
 <part name="U$10" library="microbuilder" deviceset="VIN" device=""/>
 <part name="U$11" library="microbuilder" deviceset="3.3V" device=""/>
@@
 <part name="FID2" library="microbuilder" deviceset="FIDUCIAL" device="&quot;&quot;"/>
 <part name="U$17" library="microbuilder" deviceset="VIN" device=""/>
-<part name="RTC" library="microbuilder" deviceset="SOLDERJUMPER_CLOSED" device=""/>
-<part name="U$18" library="microbuilder" deviceset="3.3V" device=""/>
+<part name="U$19" library="microbuilder" deviceset="GND" device=""/>
+<part name="U$20" library="microbuilder" deviceset="U.FL" device=""/>
+<part name="JP1" library="microbuilder" deviceset="HEADER-1X9" device="70MIL"/>
 </parts>
 <sheets>
 <sheet>
 <plain>
-<text x="134.62" y="83.82" size="1.778" layer="97">D1+R3 restrict RX input to 3.3V</text>
+<text x="134.62" y="78.74" size="1.778" layer="97">D1+R3 restrict RX input to 3.3V</text>
 </plain>
 <instances>
@@
 <instance part="U$8" gate="G$1" x="251.46" y="33.02"/>
 <instance part="U$9" gate="G$1" x="243.84" y="33.02"/>
-<instance part="JP1" gate="A" x="68.58" y="109.22" rot="R180"/>
 <instance part="U$10" gate="G$1" x="99.06" y="121.92"/>
 <instance part="U$11" gate="G$1" x="91.44" y="121.92"/>
@@
 <instance part="R3" gate="G$1" x="121.92" y="83.82" rot="R270"/>
 <instance part="U$13" gate="G$1" x="121.92" y="91.44"/>
-<instance part="B1" gate="G$1" x="104.14" y="139.7"/>
-<instance part="U$14" gate="G$1" x="93.98" y="134.62"/>
+<instance part="B1" gate="G$1" x="162.56" y="152.4" rot="R180"/>
+<instance part="U$14" gate="G$1" x="172.72" y="147.32"/>
 <instance part="FID1" gate="G$1" x="251.46" y="27.94"/>
 <instance part="FID2" gate="G$1" x="243.84" y="27.94"/>
 <instance part="U$17" gate="G$1" x="99.06" y="78.74"/>
-<instance part="RTC" gate="G$1" x="165.1" y="139.7"/>
-<instance part="U$18" gate="G$1" x="172.72" y="142.24"/>
+<instance part="U$19" gate="G$1" x="200.66" y="83.82"/>
+<instance part="U$20" gate="G$1" x="190.5" y="96.52" rot="MR0"/>
+<instance part="JP1" gate="A" x="68.58" y="106.68" rot="R180"/>
 </instances>
 <busses>
@@
 <wire x1="71.12" y1="109.22" x2="86.36" y2="109.22" width="0.1524" layer="91"/>
 <label x="76.2" y="109.22" size="1.778" layer="95"/>
-<pinref part="JP1" gate="A" pin="5"/>
+<pinref part="JP1" gate="A" pin="6"/>
 </segment>
 </net>
@@
 <wire x1="71.12" y1="101.6" x2="93.98" y2="101.6" width="0.1524" layer="91"/>
 <pinref part="U$12" gate="G$1" pin="GND"/>
-<pinref part="JP1" gate="A" pin="2"/>
-</segment>
-<segment>
-<wire x1="99.06" y1="139.7" x2="93.98" y2="139.7" width="0.1524" layer="91"/>
-<wire x1="93.98" y1="139.7" x2="93.98" y2="137.16" width="0.1524" layer="91"/>
+<pinref part="JP1" gate="A" pin="3"/>
+</segment>
+<segment>
+<wire x1="180.34" y1="99.06" x2="200.66" y2="99.06" width="0.1524" layer="91"/>
+<wire x1="200.66" y1="99.06" x2="200.66" y2="91.44" width="0.1524" layer="91"/>
+<wire x1="200.66" y1="91.44" x2="200.66" y2="88.9" width="0.1524" layer="91"/>
+<wire x1="200.66" y1="88.9" x2="200.66" y2="86.36" width="0.1524" layer="91"/>
+<wire x1="180.34" y1="116.84" x2="200.66" y2="116.84" width="0.1524" layer="91"/>
+<wire x1="200.66" y1="116.84" x2="200.66" y2="99.06" width="0.1524" layer="91"/>
+<wire x1="193.04" y1="88.9" x2="200.66" y2="88.9" width="0.1524" layer="91"/>
+<wire x1="193.04" y1="91.44" x2="200.66" y2="91.44" width="0.1524" layer="91"/>
+<junction x="200.66" y="99.06"/>
+<junction x="200.66" y="88.9"/>
+<junction x="200.66" y="91.44"/>
+<pinref part="U1" gate="G$1" pin="GND@3"/>
+<pinref part="U$19" gate="G$1" pin="GND"/>
+<pinref part="U1" gate="G$1" pin="GND@4"/>
+<pinref part="U$20" gate="G$1" pin="GND@1"/>
+<pinref part="U$20" gate="G$1" pin="GND@0"/>
+</segment>
+<segment>
+<wire x1="167.64" y1="152.4" x2="172.72" y2="152.4" width="0.1524" layer="91"/>
+<wire x1="172.72" y1="152.4" x2="172.72" y2="149.86" width="0.1524" layer="91"/>
 <pinref part="B1" gate="G$1" pin="-"/>
 <pinref part="U$14" gate="G$1" pin="GND"/>
@@
 <wire x1="71.12" y1="116.84" x2="91.44" y2="116.84" width="0.1524" layer="91"/>
 <pinref part="U$11" gate="G$1" pin="3.3V"/>
-<pinref part="JP1" gate="A" pin="8"/>
+<pinref part="JP1" gate="A" pin="9"/>
 </segment>
 <segment>
@@
 <pinref part="U1" gate="G$1" pin="VCC"/>
 </segment>
-<segment>
-<wire x1="170.18" y1="139.7" x2="172.72" y2="139.7" width="0.1524" layer="91"/>
-<wire x1="172.72" y1="139.7" x2="172.72" y2="142.24" width="0.1524" layer="91"/>
-<pinref part="RTC" gate="G$1" pin="2"/>
-<pinref part="U$18" gate="G$1" pin="3.3V"/>
-</segment>
 </net>
 <net name="ENABLE" class="0">
@@
 <wire x1="71.12" y1="114.3" x2="86.36" y2="114.3" width="0.1524" layer="91"/>
 <label x="76.2" y="114.3" size="1.778" layer="95"/>
-<pinref part="JP1" gate="A" pin="7"/>
+<pinref part="JP1" gate="A" pin="8"/>
 </segment>
 <segment>
@@
 <wire x1="99.06" y1="99.06" x2="99.06" y2="121.92" width="0.1524" layer="91"/>
 <pinref part="U$10" gate="G$1" pin="VIN"/>
-<pinref part="JP1" gate="A" pin="1"/>
+<pinref part="JP1" gate="A" pin="2"/>
 </segment>
 <segment>
@@
 </segment>
 <segment>
-<wire x1="109.22" y1="139.7" x2="121.92" y2="139.7" width="0.1524" layer="91"/>
-<label x="111.76" y="139.7" size="1.778" layer="95"/>
-<pinref part="B1" gate="G$1" pin="+"/>
-</segment>
-<segment>
 <wire x1="71.12" y1="111.76" x2="86.36" y2="111.76" width="0.1524" layer="91"/>
 <label x="76.2" y="111.76" size="1.778" layer="95"/>
-<pinref part="JP1" gate="A" pin="6"/>
-</segment>
-<segment>
-<wire x1="160.02" y1="139.7" x2="147.32" y2="139.7" width="0.1524" layer="91"/>
-<label x="147.32" y="139.7" size="1.778" layer="95"/>
-<pinref part="RTC" gate="G$1" pin="1"/>
+<pinref part="JP1" gate="A" pin="7"/>
+</segment>
+<segment>
+<wire x1="157.48" y1="152.4" x2="142.24" y2="152.4" width="0.1524" layer="91"/>
+<label x="142.24" y="152.4" size="1.778" layer="95"/>
+<pinref part="B1" gate="G$1" pin="+"/>
 </segment>
 </net>
@@
 <wire x1="71.12" y1="106.68" x2="86.36" y2="106.68" width="0.1524" layer="91"/>
 <label x="76.2" y="106.68" size="1.778" layer="95"/>
-<pinref part="JP1" gate="A" pin="4"/>
+<pinref part="JP1" gate="A" pin="5"/>
 </segment>
 </net>
@@
 <wire x1="71.12" y1="104.14" x2="86.36" y2="104.14" width="0.1524" layer="91"/>
 <label x="76.2" y="104.14" size="1.778" layer="95"/>
-<pinref part="JP1" gate="A" pin="3"/>
+<pinref part="JP1" gate="A" pin="4"/>
+</segment>
+</net>
+<net name="N$4" class="0">
+<segment>
+<wire x1="180.34" y1="96.52" x2="185.42" y2="96.52" width="0.1524" layer="91"/>
+<pinref part="U1" gate="G$1" pin="EX_ANT"/>
+<pinref part="U$20" gate="G$1" pin="SIGNAL"/>
+</segment>
+</net>
+<net name="1PPS" class="0">
+<segment>
+<wire x1="180.34" y1="101.6" x2="193.04" y2="101.6" width="0.1524" layer="91"/>
+<label x="185.42" y="101.6" size="1.778" layer="95"/>
+<pinref part="U1" gate="G$1" pin="1PPS"/>
+</segment>
+<segment>
+<wire x1="71.12" y1="96.52" x2="86.36" y2="96.52" width="0.1524" layer="91"/>
+<label x="76.2" y="96.52" size="1.778" layer="95"/>
+<pinref part="JP1" gate="A" pin="1"/>
 </segment>
 </net>
@@
 </sheet>
 </sheets>
+<errors>
+</errors>
 </schematic>
 </drawing>

Commit message: updated!
Parts:
- added D2: CUS520, microbuilder:DIODESOD-323
- C1, C2, C3: device microbuilder:CAP_CERAMIC0805 -> microbuilder:CAP_CERAMIC0805-NOOUTLINE
- D1: device adafruit:DIODESOD-323F -> microbuilder:DIODESOD-323
- FB1: device microbuilder:FERRITE0805 -> microbuilder:FERRITE-0805NO
- LED1: value FIX -> RED
- R1, R2, R3: device microbuilder:RESISTOR0805 -> microbuilder:RESISTOR0805_NOOUTLINE
- U$8, U$9: value MOUNTINGHOLE2.0 -> MOUNTINGHOLE2.5; device microbuilder:MOUNTINGHOLE2.0 -> microbuilder:MOUNTINGHOLE2.5
- U2: value RT9193-3.3 -> MIC5225-3.3
Connections:
- removed net RX_5V: D1.C, JP1.4
- new net N$1: B1.+, D2.A
- new net RX_3V: D1.A, R3.2, U1.RX
- net 3.3V: now also C1.1, C2.1; no longer C1.P$1, C2.P$1
- net GND: now also C1.2, C2.2, C3.2; no longer C1.P$2, C2.P$2, C3.P$2
- net RX: now also D1.C, JP1.4; no longer D1.A, R3.2, U1.RX
- net VBACKUP: now also D2.C; no longer B1.+
- net VIN: now also C3.1; no longer C3.P$1
Other:
- moved on the sheet: B1
